File: sprit.kicad_sch (KiCad schematic)
At the start: 14 parts, among them J1 BARREL_JACK, J2 CONN_02X05, J3 CONN_01X03, Q1 2N7002, Q2 2N7002, U1 MC7808CDTRKG, U2 SN74LV1T126

Commit message: fix supply voltage notation, add README
Other:
- note added: "10.5-18V"
- note removed: "5-18V"
Changed lines of the file:
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@@
     (effects (font (size 1.524 1.524)) (justify left bottom))
   )
-  (text "5-18V" (at 148.59 43.18 0)
+  (text "10.5-18V" (at 148.59 43.18 0)
     (effects (font (size 1.524 1.524)) (justify left bottom))
   )
